Commit message: 透過手把遙控小車以及切換模式跟緊急停止 urdf gazebo以成功導入 缺少SLAM EKF Nav2

File: src/mowerbot_description/urdf/car.xacro (robot description, xacro)
@@ -6,4 +6,6 @@
     <xacro:include filename="car_base.xacro"/>
     <xacro:include filename="car_radar.xacro"/>
+    <xacro:include filename="car_camera.xacro"/>
+    <xacro:include filename="car_imu.xacro"/>
 </robot>
 <!--輪子半徑 0.17m 車子總長約 0.95x0.46x0.46 輪胎 1kg 車體57.2kg 電池16.2kg-->

File: src/mowerbot_description/urdf/car_base.xacro (robot description, xacro)
@@ -1,21 +1,20 @@
-<!-- 底盤 -->
-<robot xmlns:xacro="http://www.ros.org/wiki/xacro">
-    <!-- 車體尺寸 -->
-    <xacro:property name="car_length" value="3.0"/>
-    <xacro:property name="car_width" value="1.5"/>
-    <xacro:property name="car_height" value="0.6"/>
-    <!-- 離地間隙 -->
+<?xml version="1.0"?>
+<robot xmlns:xacro="http://www.ros.org/wiki/xacro" name="mowerbot">
+    <xacro:property name="car_length" value="0.95"/>
+    <xacro:property name="car_width" value="0.46"/>
+    <xacro:property name="car_height" value="0.46"/>
+    <xacro:property name="car_mass" value="73.4"/>
     <xacro:property name="ground_height" value="0.2"/>
-    <!-- 包含子文件, 要在參數定義之後, 子文件才能使用父文件的参數 -->
+    <xacro:include filename="car_inertia.xacro"/>
     <xacro:include filename="car_wheels.xacro"/>
-    <!-- 顏色 -->
     <material name="yellow">
         <color rgba="0.9 0.6 0.0 0.7"/>
     </material>
-    <!-- 根坐標 -->
     <link name="map"/>
-    <!-- 底盤在map的投影點 -->
     <link name="base_footprint"/>
-    <!-- 底盤 -->
+    <joint name="footprint_to_map" type="fixed">
+        <parent link="map"/>
+        <child link="base_footprint"/>
+    </joint>
     <link name="base_link">
         <visual>
@@ -25,15 +24,32 @@
             <material name="yellow"/>
         </visual>
+        <collision>
+            <geometry>
+                <box size="${car_length} ${car_width} ${car_height}"/>
+            </geometry>
+        </collision>
+        <xacro:box_inertia m="${car_mass}" w="${car_length}" h="${car_width}" d="${car_height}" o_xyz="0 0 -0.18"/>
     </link>
-    <!-- 投影點關聯到地圖 -->
-    <joint name="footprint_to_map" type="fixed">
-        <parent link="map"/>
-        <child link="base_footprint"/>
-    </joint>
-    <!-- 底盤關聯到投影點 -->
     <joint name="base_to_footprint" type="fixed">
         <parent link="base_footprint"/>
         <child link="base_link"/>
-        <origin xyz="0.0 0.0 ${car_height / 2.0 + ground_height}"/>
+        <origin xyz="0.0 0.0 ${car_height / 2.0 + ground_height}" rpy="0 0 0"/>
     </joint>
+    <gazebo>
+        <plugin name="mowerbot_diff_drive" filename="libgazebo_ros_diff_drive.so">
+            <left_joint>left_rear_wheel_joint</left_joint>
+            <right_joint>right_rear_wheel_joint</right_joint>
+            <wheel_separation>0.58</wheel_separation>
+            <wheel_diameter>0.34</wheel_diameter>
+            <max_wheel_torque>200</max_wheel_torque> <max_wheel_acceleration>1.0</max_wheel_acceleration>
+            <command_topic>cmd_vel</command_topic>
+            <odometry_topic>odom</odometry_topic>
+            <odometry_frame>odom</odometry_frame>
+            <robot_base_frame>base_footprint</robot_base_frame>
+            <update_rate>30</update_rate>
+            <publish_odom>true</publish_odom>
+            <publish_odom_tf>true</publish_odom_tf>
+            <publish_wheel_tf>true</publish_wheel_tf>
+        </plugin>
+    </gazebo>
 </robot>

File: src/mowerbot_description/urdf/car_radar.xacro (robot description, xacro)
@@ -2,6 +2,6 @@
 <robot xmlns:xacro="http://www.ros.org/wiki/xacro">
     <!-- 雷達尺寸 -->
-    <xacro:property name="radar_radius" value="0.2"/>
-    <xacro:property name="radar_height" value="0.2"/>
+    <xacro:property name="radar_radius" value="0.1"/>
+    <xacro:property name="radar_height" value="0.1"/>
     <!-- 雷達偏移量 -->
     <xacro:property name="radar_joint_x" value="0.0"/>
@@ -27,3 +27,30 @@
         <origin xyz="${radar_joint_x} ${radar_joint_y} ${radar_joint_z}"/>
     </joint>
+    <gazebo reference="radar">
+        <material>Gazebo/Blue</material>
+        <sensor name="lidar" type="ray">
+            <always_on>true</always_on>
+            <visualize>true</visualize>
+            <update_rate>10.0</update_rate> <ray>
+                <scan>
+                    <horizontal>
+                        <samples>360</samples> <resolution>1.0</resolution>
+                        <min_angle>-3.1415926</min_angle> <max_angle>3.1415926</max_angle>  </horizontal>
+                </scan>
+                <range>
+                    <min>0.15</min> <max>12.0</max> <resolution>0.01</resolution> </range>
+                <noise>
+                    <type>gaussian</type>
+                    <mean>0.0</mean>
+                    <stddev>0.01</stddev> </noise>
+            </ray>
+            <plugin name="scan_node" filename="libgazebo_ros_ray_sensor.so">
+                <ros>
+                    <remapping>~/out:=scan</remapping>
+                </ros>
+                <output_type>sensor_msgs/LaserScan</output_type>
+                <frame_name>radar</frame_name>
+            </plugin>
+        </sensor>
+    </gazebo>
 </robot>

File: src/mowerbot_description/urdf/car_wheels.xacro (robot description, xacro)
@@ -1,65 +1,62 @@
-<!-- 車輪 -->
+<?xml version="1.0"?>
 <robot xmlns:xacro="http://www.ros.org/wiki/xacro">
-    <!-- 車輪尺寸 -->
-    <xacro:property name="wheel_radius" value="${car_height / 2.0 + wheel_joint_z + ground_height}"/>
-    <xacro:property name="wheel_width" value="0.3"/>
-    <!-- 車輪偏移量 -->
-    <xacro:property name="wheel_joint_x" value="${car_length / 2.0 - 0.4}"/>
-    <xacro:property name="wheel_joint_y" value="${car_width / 2.0 + wheel_width/ 2.0 + 0.1}"/>
-    <xacro:property name="wheel_joint_z" value="-0.2"/>
-    <!-- 颜色 -->
-    <material name="black">
-        <color rgba="0.0 0.0 0.0 0.7"/>
-    </material>
-    <!-- 車輪幾何 -->
-    <xacro:macro name="wheel_geometry" params="wheel_name">
-        <link name="${wheel_name}">
+    <xacro:include filename="car_inertia.xacro"/>
+    <xacro:property name="PI" value="3.1415926535897931"/>
+    <xacro:property name="body_length" value="0.95"/>
+    <xacro:property name="body_width" value="0.46"/>
+    <xacro:property name="body_height" value="0.46"/>
+    <xacro:property name="wheel_radius" value="0.17"/>
+    <xacro:property name="wheel_width" value="0.1"/>
+    <xacro:property name="wheel_mass" value="1.0"/>
+    <xacro:macro name="visual_wheel" params="prefix">
+        <link name="${prefix}_wheel">
             <visual>
+                <origin xyz="0 0 0" rpy="${PI/2} 0 0"/>
                 <geometry>
                     <cylinder radius="${wheel_radius}" length="${wheel_width}"/>
                 </geometry>
-                <origin rpy="${PI / 2.0} 0.0 0.0"/>
-                <material name="black"/>
+                <material name="black">
+                    <color rgba="0.1 0.1 0.1 1.0"/>
+                </material>
             </visual>
+            <collision>
+                <origin xyz="0 0 0" rpy="${PI/2} 0 0"/>
+                <geometry>
+                    <cylinder radius="${wheel_radius}" length="${wheel_width}"/>
+                </geometry>
+            </collision>
+            <xacro:cylinder_inertia m="${wheel_mass}" r="${wheel_radius}" h="${wheel_width}" o_rpy="${PI/2} 0 0"/>
         </link>
     </xacro:macro>
-    <!-- 後輪函数 -->
-    <xacro:macro name="wheel_rear_func" params="wheel_name left_flag">
-        <!-- 車輪幾何 -->
-        <xacro:wheel_geometry wheel_name="${wheel_name}"/>
-        <!-- 車輪關聯到base_link -->
-        <joint name="${wheel_name}_rolling" type="continuous">
+    <xacro:macro name="add_rear_wheel" params="prefix y_reflect">
+        <xacro:visual_wheel prefix="${prefix}_rear" />
+        <joint name="${prefix}_rear_wheel_joint" type="continuous">
             <parent link="base_link"/>
-            <child link="${wheel_name}"/>
-            <origin xyz="${-wheel_joint_x} ${wheel_joint_y * left_flag} ${wheel_joint_z}"/>
+            <child link="${prefix}_rear_wheel"/>
+            <origin xyz="-0.35 ${y_reflect * (body_width/2 + wheel_width/2 + 0.01)} -0.26" rpy="0 0 0"/>
             <axis xyz="0 1 0"/>
         </joint>
+        <gazebo reference="${prefix}_rear_wheel">
+            <mu1>2.0</mu1>      <mu2>2.0</mu2>      <kp>1000000.0</kp>  <kd>10.0</kd>  <minDepth>0.001</minDepth>     </gazebo>
     </xacro:macro>
-    <!-- 前輪函数 -->
-    <xacro:macro name="wheel_front_func" params="wheel_name left_flag">
-        <!-- 車輪幾何 -->
-        <xacro:wheel_geometry wheel_name="${wheel_name}"/>
-        <!-- 轉向節幾何 -->
-        <link name="${wheel_name}_steering_knuckle"/>
-        <!-- 轉向關聯到base_link -->
-        <joint name="${wheel_name}_turning" type="revolute">
+    <xacro:add_rear_wheel prefix="left"  y_reflect="1" />
+    <xacro:add_rear_wheel prefix="right" y_reflect="-1" />
+    <xacro:macro name="add_front_wheel" params="prefix y_reflect">
+        <xacro:visual_wheel prefix="${prefix}_front" />
+        <joint name="${prefix}_front_wheel_joint" type="continuous">
             <parent link="base_link"/>
-            <child link="${wheel_name}_steering_knuckle"/>
-            <origin xyz="${wheel_joint_x} ${wheel_joint_y * left_flag} ${wheel_joint_z}"/>
-            <axis xyz="0 0 1"/>
-            <limit effort="0.0" velocity="0.0" lower="-${PI / 6.0}" upper="${PI / 6.0}" />
-        </joint>
-        <!-- 車輪關節到轉向輪 -->
-        <joint name="${wheel_name}_rolling" type="continuous">
-            <parent link="${wheel_name}_steering_knuckle"/>
-            <child link="${wheel_name}"/>
-            <origin xyz="0 0 0"/>
+            <child link="${prefix}_front_wheel"/>
+            <origin xyz="0.35 ${y_reflect * (body_width/2 + wheel_width/2 + 0.01)} -0.26" rpy="0 0 0"/>
             <axis xyz="0 1 0"/>
         </joint>
+        <gazebo reference="${prefix}_front_wheel">
+            <mu1>0.1</mu1>
+            <mu2>0.0</mu2>
+            <kp>1000000.0</kp>
+            <kd>100.0</kd>
+            <minDepth>0.001</minDepth>
+        </gazebo>
     </xacro:macro>
-    <!-- 生成4個輪胎 -->
-    <xacro:wheel_front_func wheel_name="left_front" left_flag="1"/>
-    <xacro:wheel_front_func wheel_name="right_front" left_flag="-1"/>
-    <xacro:wheel_rear_func wheel_name="left_rear" left_flag="1"/>
-    <xacro:wheel_rear_func wheel_name="right_rear" left_flag="-1"/>
+    <xacro:add_front_wheel prefix="left"  y_reflect="1" />
+    <xacro:add_front_wheel prefix="right" y_reflect="-1" />
 </robot>
