Commit message: 階段30【A】車輛幾何單一來源化 vehicle.yaml（純重構；外接半徑改精確值 +4.467e-5 m 為唯一數值差異，完整套件 51/51）
Co-Authored-By: Claude Opus 5.5 <noreply@anthropic.com>

File: src/mowerbot_description/urdf/car.xacro (robot description, xacro)
@@ -9,3 +9,3 @@
     <xacro:include filename="car_imu.xacro"/>
 </robot>
-<!--輪子半徑 0.17m 車子總長約 0.95x0.46x0.46 輪胎 1kg 車體57.2kg 電池16.2kg-->
+<!--車輛尺寸與質量見 config/vehicle.yaml (單一來源)。輪胎 1kg 車體57.2kg 電池16.2kg-->

File: src/mowerbot_description/urdf/car_base.xacro (robot description, xacro)
@@ -1,8 +1,10 @@
 <?xml version="1.0"?>
 <robot xmlns:xacro="http://www.ros.org/wiki/xacro" name="mowerbot">
-    <xacro:property name="car_length" value="0.95"/>
-    <xacro:property name="car_width" value="0.46"/>
-    <xacro:property name="car_height" value="0.46"/>
-    <xacro:property name="car_mass" value="73.4"/>
+    <!-- 車輛幾何的單一來源：mowerbot_description/config/vehicle.yaml (階段 30) -->
+    <xacro:property name="vehicle" value="${xacro.load_yaml('$(find mowerbot_description)/config/vehicle.yaml')}"/>
+    <xacro:property name="car_length" value="${vehicle['body_length']}"/>
+    <xacro:property name="car_width" value="${vehicle['body_width']}"/>
+    <xacro:property name="car_height" value="${vehicle['body_height']}"/>
+    <xacro:property name="car_mass" value="${vehicle['mass']}"/>
     <xacro:property name="ground_height" value="0.2"/>
     <xacro:include filename="car_inertia.xacro"/>
@@ -35,6 +37,6 @@
         <left_joint>left_rear_wheel_joint</left_joint>
         <right_joint>right_rear_wheel_joint</right_joint>
-        <wheel_separation>0.58</wheel_separation>
-        <wheel_diameter>0.34</wheel_diameter>
+        <wheel_separation>${vehicle['wheel_separation']}</wheel_separation>
+        <wheel_diameter>${2 * vehicle['wheel_radius']}</wheel_diameter>
         <max_wheel_torque>200</max_wheel_torque>
         <max_wheel_acceleration>3.0</max_wheel_acceleration>

File: src/mowerbot_description/urdf/car_wheels.xacro (robot description, xacro)
@@ -3,8 +3,10 @@
     <xacro:include filename="car_inertia.xacro"/>
     <xacro:property name="PI" value="3.1415926535897931"/>
-    <xacro:property name="body_length" value="0.95"/>
-    <xacro:property name="body_width" value="0.46"/>
-    <xacro:property name="body_height" value="0.46"/>
-    <xacro:property name="wheel_radius" value="0.17"/>
+    <!-- 車體與輪子尺寸來自 vehicle.yaml (car_base.xacro 載入的 vehicle) -->
+    <xacro:property name="body_length" value="${vehicle['body_length']}"/>
+    <xacro:property name="body_width" value="${vehicle['body_width']}"/>
+    <xacro:property name="body_height" value="${vehicle['body_height']}"/>
+    <xacro:property name="wheel_radius" value="${vehicle['wheel_radius']}"/>
+    <xacro:property name="wheel_separation" value="${vehicle['wheel_separation']}"/>
     <xacro:property name="wheel_width" value="0.1"/>
     <xacro:property name="wheel_mass" value="1.0"/>
@@ -31,8 +33,12 @@
     <xacro:macro name="add_rear_wheel" params="prefix y_reflect">
         <xacro:visual_wheel prefix="${prefix}_rear" />
+        <!-- y = +-wheel_separation/2；z 讓輪子剛好著地 = wheel_radius - base_link 離地高度。
+             以前 y 是 body_width/2 + wheel_width/2 + 0.01、z 寫死 -0.26 (= 0.17 - 0.43)，
+             量測值一換就會與 diff_drive 的 wheel_separation 對不上 / 輪子懸空或陷地。
+             x = +-0.35 (軸距 0.70) 仍然寫死：vehicle.yaml 的 wheelbase 還是 TBD。 -->
         <joint name="${prefix}_rear_wheel_joint" type="continuous">
             <parent link="base_link"/>
             <child link="${prefix}_rear_wheel"/>
-            <origin xyz="-0.35 ${y_reflect * (body_width/2 + wheel_width/2 + 0.01)} -0.26" rpy="0 0 0"/>
+            <origin xyz="-0.35 ${y_reflect * wheel_separation / 2} ${wheel_radius - (car_height / 2.0 + ground_height)}" rpy="0 0 0"/>
             <axis xyz="0 1 0"/>
         </joint>
@@ -47,5 +53,5 @@
             <parent link="base_link"/>
             <child link="${prefix}_front_wheel"/>
-            <origin xyz="0.35 ${y_reflect * (body_width/2 + wheel_width/2 + 0.01)} -0.26" rpy="0 0 0"/>
+            <origin xyz="0.35 ${y_reflect * wheel_separation / 2} ${wheel_radius - (car_height / 2.0 + ground_height)}" rpy="0 0 0"/>
             <axis xyz="0 1 0"/>
         </joint>
