Commit message: 完成SLAM建圖

File: src/mowerbot_description/urdf/car_base.xacro (robot description, xacro)
@@ -11,10 +11,5 @@
         <color rgba="0.9 0.6 0.0 0.7"/>
     </material>
-    <link name="map"/>
     <link name="base_footprint"/>
-    <joint name="footprint_to_map" type="fixed">
-        <parent link="map"/>
-        <child link="base_footprint"/>
-    </joint>
     <link name="base_link">
         <visual>
@@ -37,19 +32,20 @@
     </joint>
     <gazebo>
-        <plugin name="mowerbot_diff_drive" filename="libgazebo_ros_diff_drive.so">
-            <left_joint>left_rear_wheel_joint</left_joint>
-            <right_joint>right_rear_wheel_joint</right_joint>
-            <wheel_separation>0.58</wheel_separation>
-            <wheel_diameter>0.34</wheel_diameter>
-            <max_wheel_torque>200</max_wheel_torque> <max_wheel_acceleration>1.0</max_wheel_acceleration>
-            <command_topic>cmd_vel</command_topic>
-            <odometry_topic>odom</odometry_topic>
-            <odometry_frame>odom</odometry_frame>
-            <robot_base_frame>base_footprint</robot_base_frame>
-            <update_rate>30</update_rate>
-            <publish_odom>true</publish_odom>
-            <publish_odom_tf>true</publish_odom_tf>
-            <publish_wheel_tf>true</publish_wheel_tf>
-        </plugin>
+    <plugin name="mowerbot_diff_drive" filename="libgazebo_ros_diff_drive.so">
+        <left_joint>left_rear_wheel_joint</left_joint>
+        <right_joint>right_rear_wheel_joint</right_joint>
+        <wheel_separation>0.58</wheel_separation>
+        <wheel_diameter>0.34</wheel_diameter>
+        <max_wheel_torque>200</max_wheel_torque>
+        <max_wheel_acceleration>1.0</max_wheel_acceleration>
+        <command_topic>cmd_vel</command_topic>
+        <odometry_topic>odom</odometry_topic>
+        <odometry_frame>odom</odometry_frame>
+        <robot_base_frame>base_footprint</robot_base_frame>
+        <update_rate>30</update_rate>
+        <publish_odom>true</publish_odom>
+        <publish_odom_tf>true</publish_odom_tf>
+        <publish_wheel_tf>false</publish_wheel_tf>
+    </plugin>
     </gazebo>
 </robot>
