Commit message: 接上 Nav2 與 F2C 覆蓋路徑執行，並加入自動化冒煙測試
mowerbot_action/manager.py:
  - 新增 FollowPath action client，將 F2C 產生的覆蓋路徑切成多條割草線，
    逐條送給 Nav2 執行，等 SUCCEEDED 再送下一條
  - 新增 approach 路徑：從當下位置(查 map -> base_footprint)接到第 1 條割草線起點
  - 新增 /f2c_boundary 訂閱與 /f2c_path 發布(TRANSIENT_LOCAL，供 RViz 顯示)
  - 急停時取消 goal handle 並清空佇列
  - mode 3 標籤改為「保留」，行為不變

mowerbot_planner (新套件):
  - f2c_server.cpp：Fields2Cover 服務端，吃 PolygonStamped 邊界，
    產生 swath 覆蓋路徑
  - mowerbot_interfaces/srv/GenerateCoveragePath.srv 服務介面

mowerbot_bringup:
  - 新增 nav2_params.yaml 與 navigation.launch.py
  - 新增 worlds/mow_field.world 測試場地
  - setup.py 安裝 worlds/

mowerbot_bridge:
  - joystick_yaml 更名為 joystick.yaml(原本沒有副檔名，launch 讀不到)
  - teleop.py 調整

mowerbot_description:
  - urdf 各 xacro 修正 Gazebo plugin 與 sensor 設定

test/smoke_test.py:
  - 新增可重複執行的自動化冒煙測試，涵蓋 Phase A(建置/介面)、
    B(F2C/邊界)、C(Gazebo/TF)、D(安全機制)、N(Nav2 覆蓋任務)

Co-Authored-By: Claude Opus 5 <noreply@anthropic.com>

File: src/mowerbot_description/urdf/car_base.xacro (robot description, xacro)
@@ -38,5 +38,5 @@
         <wheel_diameter>0.34</wheel_diameter>
         <max_wheel_torque>200</max_wheel_torque>
-        <max_wheel_acceleration>1.0</max_wheel_acceleration>
+        <max_wheel_acceleration>3.0</max_wheel_acceleration>
         <command_topic>cmd_vel</command_topic>
         <odometry_topic>odom</odometry_topic>

File: src/mowerbot_description/urdf/car_camera.xacro (robot description, xacro)
@@ -21,4 +21,5 @@
             <material name="red"/>
         </visual>
+        <xacro:box_inertia m="0.1" w="${camera_length}" h="${camera_width}" d="${camera_height}"/>
     </link>
     <!-- 攝像機關聯到base_link -->

File: src/mowerbot_description/urdf/car_imu.xacro (robot description, xacro)
@@ -10,4 +10,5 @@
             </material>
         </visual>
+        <xacro:box_inertia m="0.02" w="0.02" h="0.02" d="0.02"/>
     </link>
     <joint name="imu_joint" type="fixed">

File: src/mowerbot_description/urdf/car_radar.xacro (robot description, xacro)
@@ -7,5 +7,7 @@
     <xacro:property name="radar_joint_x" value="0.0"/>
     <xacro:property name="radar_joint_y" value="0.0"/>
-    <xacro:property name="radar_joint_z" value="${car_height / 2.0 + radar_height / 2.0}"/>
+    <!-- 抬高到 0.45：雷達佔據 z = 0.40 ~ 0.50，完全高於相機頂端的 0.31，
+         避免 360 度掃描一直掃到車頭前方 0.455m 的相機 -->
+    <xacro:property name="radar_joint_z" value="0.45"/>
     <!-- 顏色 -->
     <material name="blue">
@@ -20,4 +22,5 @@
             <material name="blue"/>
         </visual>
+        <xacro:cylinder_inertia m="0.2" r="${radar_radius}" h="${radar_height}"/>
     </link>
     <!-- 雷達關聯到base_link -->

Commit message: 階段38 實機前整備：平台換 XLK X2RS（車輛幾何/URDF 依實測值、前輪改萬向輪、vehicle_geometry.py 推導 headland 與淨空門檻）、wheeltec 驅動、deploy 部署腳本、量測工單與現場檢查表、joy_tester 改為一般目錄、stage29_lawn 參考地圖
Co-Authored-By: Claude Opus 5.5 <noreply@anthropic.com>

File: src/mowerbot_description/urdf/car_base.xacro (robot description, xacro)
@@ -1,13 +1,38 @@
 <?xml version="1.0"?>
 <robot xmlns:xacro="http://www.ros.org/wiki/xacro" name="mowerbot">
-    <!-- 車輛幾何的單一來源：mowerbot_description/config/vehicle.yaml (階段 30) -->
+    <!-- 車輛幾何的單一來源：mowerbot_description/config/vehicle.yaml (階段 30)。
+         衍生量 (軸距、前後伸出量、側向半寬) 不在 xacro 裡重算，由
+         vehicle_geometry.xacro_mappings() 當 xacro 參數傳進來 (階段 38)，公式只有一份。
+         直接跑 xacro 而沒有帶這些參數時會失敗，這是刻意的。 -->
     <xacro:property name="vehicle" value="${xacro.load_yaml('$(find mowerbot_description)/config/vehicle.yaml')}"/>
-    <xacro:property name="car_length" value="${vehicle['body_length']}"/>
-    <xacro:property name="car_width" value="${vehicle['body_width']}"/>
-    <xacro:property name="car_height" value="${vehicle['body_height']}"/>
+    <xacro:arg name="wheelbase" default=""/>
+    <xacro:arg name="front_extent" default=""/>
+    <xacro:arg name="rear_extent" default=""/>
+    <xacro:arg name="lateral_half_extent" default=""/>
+    <xacro:arg name="lidar_z" default=""/>
+    <xacro:arg name="engine_center_x" default=""/>
+    <xacro:property name="wheelbase" value="${float('$(arg wheelbase)')}"/>
+    <xacro:property name="front_extent" value="${float('$(arg front_extent)')}"/>
+    <xacro:property name="rear_extent" value="${float('$(arg rear_extent)')}"/>
+    <xacro:property name="lateral_half_extent" value="${float('$(arg lateral_half_extent)')}"/>
+    <!-- 光達相對 base_link 的高度 = lidar_z_ground - rear_wheel_radius；引擎中心 x = 刀盤中心 (曲軸同心) -->
+    <xacro:property name="lidar_z" value="${float('$(arg lidar_z)')}"/>
+    <xacro:property name="engine_center_x" value="${float('$(arg engine_center_x)')}"/>
+    <!-- base_link = 後輪軸中心 (階段 38)。前輪是腳輪，純差速的瞬時旋轉中心就在這裡。
+         base_footprint 是它在地面的投影，base_link 離地 rear_wheel_radius。 -->
+    <xacro:property name="rear_r" value="${vehicle['rear_wheel_radius']}"/>
     <xacro:property name="car_mass" value="${vehicle['mass']}"/>
-    <xacro:property name="ground_height" value="0.2"/>
+    <!-- 車體方塊：前後涵蓋整個 footprint (-rear_extent ~ front_extent)，左右 ±lateral_half_extent，
+         上下從 body_ground_clearance 到 body_height (都是離地)。
+         camera / imu 的位置以它為準 (car_camera.xacro / car_imu.xacro)。 -->
+    <xacro:property name="car_length" value="${front_extent + rear_extent}"/>
+    <xacro:property name="car_width" value="${2.0 * lateral_half_extent}"/>
+    <xacro:property name="body_center_x" value="${(front_extent - rear_extent) / 2.0}"/>
+    <xacro:property name="body_bottom_z" value="${vehicle['body_ground_clearance'] - rear_r}"/>
+    <xacro:property name="body_top_z" value="${vehicle['body_height'] - rear_r}"/>
+    <xacro:property name="car_height" value="${body_top_z - body_bottom_z}"/>
     <xacro:include filename="car_inertia.xacro"/>
     <xacro:include filename="car_wheels.xacro"/>
+    <xacro:include filename="car_engine.xacro"/>
     <material name="yellow">
         <color rgba="0.9 0.6 0.0 0.7"/>
@@ -16,4 +41,5 @@
     <link name="base_link">
         <visual>
+            <origin xyz="${body_center_x} 0 ${(body_bottom_z + body_top_z) / 2.0}"/>
             <geometry>
                 <box size="${car_length} ${car_width} ${car_height}"/>
@@ -21,15 +47,36 @@
             <material name="yellow"/>
         </visual>
+        <!-- 光達掃描面不得落在這個方塊的高度範圍內 (vehicle_geometry.py 啟動斷言)，
+             否則模擬中車體會遮蔽自身光達。 -->
         <collision>
+            <origin xyz="${body_center_x} 0 ${(body_bottom_z + body_top_z) / 2.0}"/>
             <geometry>
                 <box size="${car_length} ${car_width} ${car_height}"/>
             </geometry>
         </collision>
-        <xacro:box_inertia m="${car_mass}" w="${car_length}" h="${car_width}" d="${car_height}" o_xyz="0 0 -0.18"/>
+        <!-- 質心 (com_x, com_height) 是暫定值，決定後輪 / 腳輪的載重分配 = 模擬裡的牽引力 -->
+        <xacro:box_inertia m="${car_mass}" w="${car_length}" h="${car_width}" d="${car_height}"
+                           o_xyz="${vehicle['com_x']} 0 ${vehicle['com_height'] - rear_r}"/>
     </link>
     <joint name="base_to_footprint" type="fixed">
         <parent link="base_footprint"/>
         <child link="base_link"/>
-        <origin xyz="0.0 0.0 ${car_height / 2.0 + ground_height}" rpy="0 0 0"/>
+        <origin xyz="0.0 0.0 ${rear_r}" rpy="0 0 0"/>
+    </joint>
+    <!-- 刀片 (階段 38)：後輪軸前方 blade_offset_x，貼地。只發 TF (覆蓋率用刀片軌跡算)，沒有碰撞。 -->
+    <link name="blade_link">
+        <visual>
+            <geometry>
+                <cylinder radius="${vehicle['blade_width'] / 2.0}" length="0.005"/>
+            </geometry>
+            <material name="grey">
+                <color rgba="0.5 0.5 0.5 0.4"/>
+            </material>
+        </visual>
+    </link>
+    <joint name="blade_joint" type="fixed">
+        <parent link="base_link"/>
+        <child link="blade_link"/>
+        <origin xyz="${vehicle['blade_offset_x']} 0 ${-rear_r}" rpy="0 0 0"/>
     </joint>
     <gazebo>
@@ -38,5 +85,5 @@
         <right_joint>right_rear_wheel_joint</right_joint>
         <wheel_separation>${vehicle['wheel_separation']}</wheel_separation>
-        <wheel_diameter>${2 * vehicle['wheel_radius']}</wheel_diameter>
+        <wheel_diameter>${2 * rear_r}</wheel_diameter>
         <max_wheel_torque>200</max_wheel_torque>
         <max_wheel_acceleration>3.0</max_wheel_acceleration>

File: src/mowerbot_description/urdf/car_camera.xacro (robot description, xacro)
@@ -6,7 +6,8 @@
     <xacro:property name="camera_height" value="0.08"/>
     <!-- 攝像機偏移量 -->
-    <xacro:property name="camera_joint_x" value="${car_length / 2.0 - 0.02}"/>
+    <!-- 車頭、車體方塊頂面上 (階段 38：以 car_base.xacro 的車體方塊為準，base_link 在後輪軸) -->
+    <xacro:property name="camera_joint_x" value="${front_extent - 0.02}"/>
     <xacro:property name="camera_joint_y" value="0.0"/>
-    <xacro:property name="camera_joint_z" value="${car_height / 2.0 + camera_height / 2.0}"/>
+    <xacro:property name="camera_joint_z" value="${body_top_z + camera_height / 2.0}"/>
     <!-- 顏色 -->
     <material name="red">

File: src/mowerbot_description/urdf/car_imu.xacro (robot description, xacro)
@@ -15,5 +15,6 @@
         <parent link="base_link"/>
         <child link="imu_link"/>
-        <origin xyz="0 0 ${car_height / 2.0}" rpy="0 0 0"/>
+        <!-- 車體方塊頂面中央 (階段 38：base_link 在後輪軸，車體中心在 body_center_x) -->
+        <origin xyz="${body_center_x} 0 ${body_top_z}" rpy="0 0 0"/>
     </joint>
     <gazebo reference="imu_link">

File: src/mowerbot_description/urdf/car_radar.xacro (robot description, xacro)
@@ -4,10 +4,12 @@
     <xacro:property name="radar_radius" value="0.1"/>
     <xacro:property name="radar_height" value="0.1"/>
-    <!-- 雷達偏移量 -->
-    <xacro:property name="radar_joint_x" value="0.0"/>
+    <!-- 雷達偏移量 (相對 base_link = 後輪軸中心)。階段 38：
+         x = vehicle.yaml lidar_x (measured_coarse 0.30 ± 0.08，量測基準點未確認)
+         z = lidar_z_ground - rear_wheel_radius (lidar_z_ground 0.55 是 provisional，未量測)
+         實車由 allow_provisional 閘門擋住，模擬放行。量測任務見 docs/measurement_worklist.md。
+         (階段 37 以前是舊 base_link (車體中心) 上方 0.45 m，用來避開相機頂端) -->
+    <xacro:property name="radar_joint_x" value="${vehicle['lidar_x']}"/>
     <xacro:property name="radar_joint_y" value="0.0"/>
-    <!-- 抬高到 0.45：雷達佔據 z = 0.40 ~ 0.50，完全高於相機頂端的 0.31，
-         避免 360 度掃描一直掃到車頭前方 0.455m 的相機 -->
-    <xacro:property name="radar_joint_z" value="0.45"/>
+    <xacro:property name="radar_joint_z" value="${lidar_z}"/>
     <!-- 顏色 -->
     <material name="blue">

File: src/mowerbot_description/urdf/car_wheels.xacro (robot description, xacro)
@@ -3,18 +3,23 @@
     <xacro:include filename="car_inertia.xacro"/>
     <xacro:property name="PI" value="3.1415926535897931"/>
-    <!-- 車體與輪子尺寸來自 vehicle.yaml (car_base.xacro 載入的 vehicle) -->
-    <xacro:property name="body_length" value="${vehicle['body_length']}"/>
-    <xacro:property name="body_width" value="${vehicle['body_width']}"/>
-    <xacro:property name="body_height" value="${vehicle['body_height']}"/>
-    <xacro:property name="wheel_radius" value="${vehicle['wheel_radius']}"/>
+    <!-- 輪子尺寸來自 vehicle.yaml (car_base.xacro 載入的 vehicle)。
+         階段 38：XLK X2RS = 後兩輪差速驅動 + 前兩個腳輪 (照片確認，可自由轉向)。
+         階段 37 以前前輪建成固定方向的從動輪，原地旋轉時前輪被迫側滑，
+         摩擦 mu >= 1.0 就完全轉不動 (報告 30.4) —— 那是建模假象，不是物理限制。 -->
+    <xacro:property name="rear_wheel_radius" value="${vehicle['rear_wheel_radius']}"/>
+    <xacro:property name="rear_wheel_width" value="${vehicle['rear_wheel_width']}"/>
     <xacro:property name="wheel_separation" value="${vehicle['wheel_separation']}"/>
-    <xacro:property name="wheel_width" value="0.1"/>
+    <xacro:property name="front_wheel_radius" value="${vehicle['front_wheel_radius']}"/>
+    <xacro:property name="front_wheel_width" value="${vehicle['front_wheel_width']}"/>
+    <xacro:property name="caster_track" value="${vehicle['caster_track']}"/>
+    <xacro:property name="caster_trail" value="${vehicle['caster_trail']}"/>
     <xacro:property name="wheel_mass" value="1.0"/>
-    <xacro:macro name="visual_wheel" params="prefix">
-        <link name="${prefix}_wheel">
+    <!-- ================= 後輪 (驅動) ================= -->
+    <xacro:macro name="add_rear_wheel" params="prefix y_reflect">
+        <link name="${prefix}_rear_wheel">
             <visual>
                 <origin xyz="0 0 0" rpy="${PI/2} 0 0"/>
                 <geometry>
-                    <cylinder radius="${wheel_radius}" length="${wheel_width}"/>
+                    <cylinder radius="${rear_wheel_radius}" length="${rear_wheel_width}"/>
                 </geometry>
                 <material name="black">
@@ -25,20 +30,14 @@
                 <origin xyz="0 0 0" rpy="${PI/2} 0 0"/>
                 <geometry>
-                    <cylinder radius="${wheel_radius}" length="${wheel_width}"/>
+                    <cylinder radius="${rear_wheel_radius}" length="${rear_wheel_width}"/>
                 </geometry>
             </collision>
-            <xacro:cylinder_inertia m="${wheel_mass}" r="${wheel_radius}" h="${wheel_width}" o_rpy="${PI/2} 0 0"/>
+            <xacro:cylinder_inertia m="${wheel_mass}" r="${rear_wheel_radius}" h="${rear_wheel_width}" o_rpy="${PI/2} 0 0"/>
         </link>
-    </xacro:macro>
-    <xacro:macro name="add_rear_wheel" params="prefix y_reflect">
-        <xacro:visual_wheel prefix="${prefix}_rear" />
-        <!-- y = +-wheel_separation/2；z 讓輪子剛好著地 = wheel_radius - base_link 離地高度。
-             以前 y 是 body_width/2 + wheel_width/2 + 0.01、z 寫死 -0.26 (= 0.17 - 0.43)，
-             量測值一換就會與 diff_drive 的 wheel_separation 對不上 / 輪子懸空或陷地。
-             x = +-0.35 (軸距 0.70) 仍然寫死：vehicle.yaml 的 wheelbase 還是 TBD。 -->
+        <!-- base_link 就在後輪軸中心：x = 0、z = 0，y = ±wheel_separation/2 -->
         <joint name="${prefix}_rear_wheel_joint" type="continuous">
             <parent link="base_link"/>
             <child link="${prefix}_rear_wheel"/>
-            <origin xyz="-0.35 ${y_reflect * wheel_separation / 2} ${wheel_radius - (car_height / 2.0 + ground_height)}" rpy="0 0 0"/>
+            <origin xyz="0 ${y_reflect * wheel_separation / 2} 0" rpy="0 0 0"/>
             <axis xyz="0 1 0"/>
         </joint>
@@ -48,15 +47,50 @@
     <xacro:add_rear_wheel prefix="left"  y_reflect="1" />
     <xacro:add_rear_wheel prefix="right" y_reflect="-1" />
-    <xacro:macro name="add_front_wheel" params="prefix y_reflect">
-        <xacro:visual_wheel prefix="${prefix}_front" />
-        <joint name="${prefix}_front_wheel_joint" type="continuous">
+    <!-- ================= 前輪 (腳輪) ================= -->
+    <!-- 每側兩個關節：
+           caster_swivel_joint  continuous，繞 z 軸 (垂直)，自由轉向
+           caster_roll_joint    continuous，繞 y 軸，滾動
+         轉軸 (swivel) 在滾動軸前方 caster_trail (後傾偏移 0.02 m)：輪子拖在轉軸後面才會自動回正，
+         沒有這段偏移 Gazebo 裡腳輪會抖。【caster_trail 是建模值，不是實測值】。
+         滾動軸位置：x = wheelbase (前輪最前凸點 = wheelbase + front_wheel_radius = front_extent)，
+         離地 front_wheel_radius。轉軸高度取滾動軸上方 front_wheel_radius (叉架高度，建模值)。
+         腳輪接地摩擦低 (mu 0.1 / mu2 0.05)：它只承重，不提供牽引。 -->
+    <xacro:macro name="add_caster" params="prefix y_reflect">
+        <link name="${prefix}_caster_swivel">
+            <xacro:cylinder_inertia m="0.2" r="0.02" h="0.02"/>
+        </link>
+        <joint name="${prefix}_caster_swivel_joint" type="continuous">
             <parent link="base_link"/>
+            <child link="${prefix}_caster_swivel"/>
+            <origin xyz="${wheelbase + caster_trail} ${y_reflect * caster_track / 2} ${front_wheel_radius - rear_r + front_wheel_radius}" rpy="0 0 0"/>
+            <axis xyz="0 0 1"/>
+        </joint>
+        <link name="${prefix}_front_wheel">
+            <visual>
+                <origin xyz="0 0 0" rpy="${PI/2} 0 0"/>
+                <geometry>
+                    <cylinder radius="${front_wheel_radius}" length="${front_wheel_width}"/>
+                </geometry>
+                <material name="black">
+                    <color rgba="0.1 0.1 0.1 1.0"/>
+                </material>
+            </visual>
+            <collision>
+                <origin xyz="0 0 0" rpy="${PI/2} 0 0"/>
+                <geometry>
+                    <cylinder radius="${front_wheel_radius}" length="${front_wheel_width}"/>
+                </geometry>
+            </collision>
+            <xacro:cylinder_inertia m="${wheel_mass}" r="${front_wheel_radius}" h="${front_wheel_width}" o_rpy="${PI/2} 0 0"/>
+        </link>
+        <joint name="${prefix}_caster_roll_joint" type="continuous">
+            <parent link="${prefix}_caster_swivel"/>
             <child link="${prefix}_front_wheel"/>
-            <origin xyz="0.35 ${y_reflect * wheel_separation / 2} ${wheel_radius - (car_height / 2.0 + ground_height)}" rpy="0 0 0"/>
+            <origin xyz="${-caster_trail} 0 ${-front_wheel_radius}" rpy="0 0 0"/>
             <axis xyz="0 1 0"/>
         </joint>
         <gazebo reference="${prefix}_front_wheel">
             <mu1>0.1</mu1>
-            <mu2>0.0</mu2>
+            <mu2>0.05</mu2>
             <kp>1000000.0</kp>
             <kd>100.0</kd>
@@ -64,5 +98,5 @@
         </gazebo>
     </xacro:macro>
-    <xacro:add_front_wheel prefix="left"  y_reflect="1" />
-    <xacro:add_front_wheel prefix="right" y_reflect="-1" />
+    <xacro:add_caster prefix="left"  y_reflect="1" />
+    <xacro:add_caster prefix="right" y_reflect="-1" />
 </robot>
